File: kicad/kicad.kicad_pcb (KiCad board)
At the start: 2 copper layers, 352.5 x 100 mm, 226 parts, among them SW1 RotaryEncoder_Switch, SW10 SW_Push, SW11 SW_Push, SW12 SW_Push, SW13 SW_Push, SW14 SW_Push, SW15 SW_Push, SW16 SW_Push, SW17 SW_Push, SW18 SW_Push, SW19 SW_Push, SW2 SW_Push, SW20 SW_Push, SW21 SW_Push, SW22 SW_Push, SW23 SW_Push, SW24 SW_Push, SW25 SW_Push, SW26 SW_Push, SW27 SW_Push, SW28 SW_Push, SW29 SW_Push, SW3 SW_Push, SW30 SW_Push, SW31 SW_Push, SW32 SW_Push, SW33 SW_Push, SW34 SW_Push, SW35 SW_Push, SW36 SW_Push, SW37 SW_Push, SW38 SW_Push, SW39 SW_Push, SW4 SW_Push, SW40 SW_Push, SW41 SW_Push, SW42 SW_Push, SW43 SW_Push, SW44 SW_Push, SW45 SW_Push, SW46 SW_Push, SW47 SW_Push, SW48 SW_Push, SW49 SW_Push, SW5 SW_Push, SW50 SW_Push, SW51 SW_Push, SW52 SW_Push, SW53 SW_Push, SW54 SW_Push, SW55 SW_Push, SW56 SW_Push, SW57 SW_Push, SW58 SW_Push, SW59 SW_Push, SW6 SW_Push, SW60 SW_Push, SW61 SW_Push, SW62 SW_Push, SW63 SW_Push, SW64 SW_Push, SW65 SW_Push, SW66 SW_Push, SW67 SW_Push, SW68 SW_Push, SW69 SW_Push, SW7 SW_Push, SW8 SW_Push, SW9 SW_Push, U1 MCP23017x-x-SS, U2 XIAO-nRF52840-SMD, U3 MCP23017x-x-SS, U4 XIAO-nRF52840-SMD

Commit message: routing left side of pcb
Parts:
- D106, D107, D108, D109, D110, D111, D112, D113, D114, D115, D116, D117, D118, D119, D120, D121, D122, D123, D124, D125, D126, D127, D128, D129, D130, D131, D132, D133, D134, D135, D136, D137, D138, D37, D38, D39, D40, D41, D42, D43, D44, D45, D46, D47, D48, D49, D50, D51, D52, D53, D54, D55, D56, D57, D58, D59, D60, D61, D62, D63, D64, D65, D66, D67, D68, D69, D70, D71, D72, D73: moved to B.Cu
- moved D71 0.56 mm to (150.3, 164.5), turned to 180 degrees
- turned D106 to 180 degrees
- turned D107 to 180 degrees
- turned D108 to 180 degrees
- turned D109 to 180 degrees
- turned D110 to 180 degrees
- turned D111 to 180 degrees
- turned D112 to 180 degrees
- turned D113 to 180 degrees
- turned D114 to 180 degrees
- turned D115 to 180 degrees
- turned D116 to 180 degrees
- turned D117 to 180 degrees
- turned D118 to 180 degrees
- turned D119 to 180 degrees
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Routing:
- net /LEFT/COL1: track 0.00 -> 443.2 mm, vias 0 -> 2
- net /LEFT/COL2: track 0.00 -> 429.0 mm, vias 0 -> 1
- net /LEFT/COL3: track 0.00 -> 401.4 mm, vias 0 -> 1
- net /LEFT/ROW1: track 0.00 -> 397.0 mm, vias 0 -> 3
- net /LEFT/ROW5: track 0.00 -> 378.9 mm, vias 0 -> 10
- net /LEFT/ROW4: track 0.00 -> 366.9 mm, vias 0 -> 8
- net /LEFT/COL5: track 0.00 -> 330.2 mm, vias 0 -> 3
- net /LEFT/ROW3: track 0.00 -> 314.9 mm, vias 0 -> 6
- net /LEFT/COL4: track 0.00 -> 295.3 mm, vias 0 -> 4
- net /LEFT/ROW2: track 0.00 -> 277.3 mm, vias 0 -> 6
- net /LEFT/COL0: track 0.00 -> 224.3 mm, vias 0 -> 2
- net /LEFT/ROW0: track 0.00 -> 211.7 mm, vias 0 -> 3
- net Net-(D44-DIN): track 0.00 -> 181.1 mm, vias 0 -> 2
- net /LEFT/BT_PIN: track 0.00 -> 138.7 mm
- net /LEFT/ES: track 0.00 -> 113.8 mm, vias 0 -> 1
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- added copper zone on F.Cu, net GND

Commit message: Completed routing left side and started working on right side routing
Routing:
- net Net-(D53-DOUT): track 0.00 -> 414.5 mm, vias 0 -> 6
- net /RIGHT/COL0: track 0.00 -> 370.0 mm
- net /RIGHT/ROW0: track 0.00 -> 352.8 mm, vias 0 -> 10
- net Net-(D55-DOUT): track 0.00 -> 335.6 mm, vias 0 -> 4
- net /RIGHT/COL1: track 0.00 -> 333.5 mm
- net Net-(D52-DOUT): track 0.00 -> 329.8 mm, vias 0 -> 3
- net Net-(D67-DIN): track 0.00 -> 326.7 mm, vias 0 -> 8
- net /RIGHT/COL2: track 0.00 -> 312.1 mm
- net /RIGHT/ROW1: track 0.00 -> 304.2 mm, vias 0 -> 10
- net /RIGHT/ROW4: track 0.00 -> 294.6 mm, vias 0 -> 4
- net /RIGHT/COL3: track 0.00 -> 273.2 mm, vias 0 -> 2
- net /RIGHT/ROW2: track 0.00 -> 254.0 mm, vias 0 -> 8
- net /LEFT/COL4: track 295.3 -> 512.8 mm, vias 4 -> 11
- net Net-(D44-DIN): track 181.1 -> 391.7 mm, vias 2 -> 1
- net /RIGHT/ROW7: track 0.00 -> 206.0 mm, vias 0 -> 5
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- added copper zone on F.Cu, net +3.3V
- added copper zone on B.Cu, net GND
- removed copper zone on F.Cu, net GND

Commit message: right half routing done
Routing:
- net /RIGHT/ROW7: track 206.0 -> 484.6 mm, vias 5 -> 15
- net /RIGHT/ROW0: track 352.8 -> 585.8 mm, vias 10 -> 18
- net /RIGHT/ROW1: track 304.2 -> 486.5 mm, vias 10 -> 20
- net /RIGHT/ROW2: track 254.0 -> 427.4 mm, vias 8 -> 16
- net /RIGHT/ROW5: track 142.4 -> 308.0 mm, vias 0 -> 9
- net Net-(D125-DIN): track 0.00 -> 142.6 mm
- net /RIGHT/ROW3: track 155.0 -> 289.4 mm, vias 2 -> 5
- net /LEFT/ROW0: track 211.7 -> 327.9 mm, vias 3 -> 13
- net Net-(D131-DOUT): track 0.00 -> 114.1 mm
- net Net-(D135-DOUT): track 0.00 -> 104.2 mm, vias 0 -> 2
- net +3.3V: track 6.89 -> 110.3 mm, vias 40 -> 89
- net /RIGHT/ROW4: track 294.6 -> 383.0 mm, vias 4 -> 8
- net Net-(D137-DIN): track 0.00 -> 65.7 mm, vias 0 -> 2
- net /RIGHT/COL3: track 273.2 -> 336.9 mm
- net Net-(D134-DOUT): track 0.00 -> 46.7 mm
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